Commit message: Include ros2_controller to control the wheels of the robot and visualize the joints movement in Gazebo and Rviz. Update readme

File: robotino_description/urdf/robotino.urdf (robot description, URDF)
Before this commit: robot robotino, 5 links, 4 joints
Joints:
- removed joint fixed
- added joint base_joint: type fixed, parent base_footprint, child base_link, origin xyz=0 0 0 rpy=0 0 0

Commit message: Movement visualitation in Gazebo and RViz with ros_plannar_move plugin

File: robotino_description/urdf/robotino.urdf (robot description, URDF)
Before this commit: robot robotino, 5 links, 4 joints
Joints:
- joint wheel0_joint: type continuous -> fixed
- joint wheel1_joint: type continuous -> fixed
- joint wheel2_joint: type continuous -> fixed
