Commit message: Fixed imu and lidar

File: robotino_description/urdf/common_properties.xacro (robot description, xacro)
@@ -7,3 +7,6 @@
         <color rgba="0.5 0.5 0.5 1" />
     </material>
+    <material name="blue">
+        <color rgba="0 0 1 1" />
+    </material>
 </robot>

File: robotino_description/urdf/lidar.xacro (robot description, xacro)
@@ -62,5 +62,5 @@
                 <scan>
                     <horizontal>
-                        <samples>686</samples>
+                        <samples>683</samples>
                         <min_angle>-2.094395102</min_angle>
                         <max_angle>2.094395102</max_angle>
@@ -74,9 +74,7 @@
             </ray>
             <plugin name="laser_controller" filename="libgazebo_ros_ray_sensor.so">
-                <!--
                 <ros>
                     <argument>~/out:=scan</argument>
                 </ros>
-                -->
                 <output_type>sensor_msgs/LaserScan</output_type>
                 <frame_name>lidar_link</frame_name>

File: robotino_description/urdf/robotino.urdf.xacro (robot description, xacro)
@@ -5,3 +5,4 @@
     <xacro:include filename="mobile_base_gazebo.xacro" />
     <xacro:include filename="lidar.xacro" />
+    <xacro:include filename="imu.xacro" />
 </robot>
